Commit message: Multi-agent control active

File: urdf/turtlebot4_hat.urdf.xacro (robot description, xacro)
@@ -17,5 +17,5 @@
     <visual>
       <geometry>
-        <cylinder radius="0.11" length="0.02"/>
+        <cylinder radius="0.12" length="0.02"/>
       </geometry>
       <material name="hat_material">
@@ -27,5 +27,5 @@
     <parent link="shell_link"/>
     <child link="hat_link"/>
-    <origin xyz="0 0 0.12" rpy="0 0 0"/>
+    <origin xyz="0 0 0.26" rpy="0 0 0"/>
   </joint>
   <!-- Ignition/Gazebo material (this is what the sim renders) -->
